Commit message: sync changes

File: turtlebot3_description/urdf/turtlebot3_waffle_pi.gazebo.xacro (robot description, xacro)
@@ -105,5 +105,5 @@
     <material>Gazebo/FlatBlack</material>
     <sensor type="ray" name="lds_lfcd_sensor">
-      <pose>0 0 0 0 0 0</pose>
+      <pose>0 0 -2.5 0 0 0</pose>
       <visualize>$(arg laser_visual)</visualize>
       <update_rate>5</update_rate>

File: turtlebot3_description/urdf/turtlebot3_waffle_pi_for_open_manipulator.gazebo.xacro (robot description, xacro)
@@ -4,13 +4,14 @@
   <xacro:arg name="camera_visual" default="false"/>
   <xacro:arg name="imu_visual"    default="false"/>
+  <xacro:arg name="tf_prefix"    default=""/>
   <gazebo reference="base_link">
     <material>Gazebo/DarkGrey</material>
   </gazebo>
   <gazebo reference="wheel_left_link">
-    <mu1>10000</mu1>
-    <mu2>10000</mu2>
-    <kp>500000.0</kp>
-    <kd>10.0</kd>
-    <minDepth>0.001</minDepth>
+    <mu1>1000000000</mu1>
+    <mu2>1000000000</mu2>
+    <kp>500000000.0</kp>
+    <kd>10000.0</kd>
+    <minDepth>0.0005</minDepth>
     <maxVel>0.1</maxVel>
     <fdir1>1 0 0</fdir1>
@@ -18,9 +19,9 @@
   </gazebo>
   <gazebo reference="wheel_right_link">
-    <mu1>10000</mu1>
-    <mu2>10000</mu2>
-    <kp>500000.0</kp>
-    <kd>10.0</kd>
-    <minDepth>0.001</minDepth>
+    <mu1>1000000000</mu1>
+    <mu2>1000000000</mu2>
+    <kp>500000000.0</kp>
+    <kd>10000.0</kd>
+    <minDepth>0.0005</minDepth>
     <maxVel>0.1</maxVel>
     <fdir1>1 0 0</fdir1>
@@ -52,12 +53,13 @@
     <material>Gazebo/Grey</material>
   </gazebo>
+  <xacro:property name="ns" value="turtlebot3" />
   <gazebo>
     <plugin name="turtlebot3_waffle_pi_controller" filename="libgazebo_ros_diff_drive.so">
       <commandTopic>cmd_vel</commandTopic>
       <odometryTopic>odom</odometryTopic>
-      <odometryFrame>odom</odometryFrame>
+      <odometryFrame>$(arg tf_prefix)/odom</odometryFrame>
       <odometrySource>world</odometrySource>
       <publishOdomTF>true</publishOdomTF>
-      <robotBaseFrame>base_footprint</robotBaseFrame>
+      <robotBaseFrame>$(arg tf_prefix)/base_footprint</robotBaseFrame>
       <publishWheelTF>false</publishWheelTF>
       <publishTf>true</publishTf>
@@ -78,5 +80,5 @@
       <alwaysOn>true</alwaysOn>
       <bodyName>imu_link</bodyName>
-      <frameName>imu_link</frameName>
+      <frameName>$(arg tf_prefix)/imu_link</frameName>
       <topicName>imu</topicName>
       <serviceName>imu_service</serviceName>
@@ -105,7 +107,7 @@
     <material>Gazebo/FlatBlack</material>
     <sensor type="ray" name="lds_lfcd_sensor">
-      <pose>0 0 0 0 0 0</pose>
-      <visualize>$(arg laser_visual)</visualize>
-      <update_rate>5</update_rate>
+      <pose>0 0 -0.28 0 0 0</pose>
+      <visualize>false</visualize>
+      <update_rate>10</update_rate>
       <ray>
         <scan>
@@ -118,7 +120,7 @@
         </scan>
         <range>
-          <min>0.120</min>
+          <min>0.40</min>
           <max>3.5</max>
-          <resolution>0.015</resolution>
+          <resolution>0.01</resolution>
         </range>
         <noise>
@@ -130,5 +132,5 @@
       <plugin name="gazebo_ros_lds_lfcd_controller" filename="libgazebo_ros_laser.so">
         <topicName>scan</topicName>
-        <frameName>base_scan</frameName>
+        <frameName>$(arg tf_prefix)/base_scan</frameName>
       </plugin>
     </sensor>

File: turtlebot3_description/urdf/turtlebot3_waffle_pi_for_open_manipulator.urdf.xacro (robot description, xacro)
@@ -1,5 +1,7 @@
 <?xml version="1.0" ?>
 <robot name="turtlebot3_waffle_pi_for_open_manipulator" xmlns:xacro="http://ros.org/wiki/xacro">
+  <xacro:arg name="tf_prefix" default=""/>
   <xacro:include filename="$(find turtlebot3_description)/urdf/common_properties.xacro"/>
+  <!-- Include the main turtlebot3 xacro file -->
   <xacro:include filename="$(find turtlebot3_description)/urdf/turtlebot3_waffle_pi_for_open_manipulator.gazebo.xacro"/>
   <link name="base_footprint"/>
@@ -56,8 +58,8 @@
     <inertial>
       <origin xyz="0 0 0" />
-      <mass value="2.8498940e-02" />
-      <inertia ixx="1.1175580e-05" ixy="-4.2369783e-11" ixz="-5.9381719e-09"
-               iyy="1.1192413e-05" iyz="-1.4400107e-11"
-               izz="2.0712558e-05" />
+      <mass value="2.8498940" />
+      <inertia ixx="1.1175580e-03" ixy="-4.2369783e-09" ixz="-5.9381719e-07"
+               iyy="1.1192413e-03" iyz="-1.4400107e-09"
+               izz="2.0712558e-03" />
       </inertial>
   </link>
@@ -84,8 +86,8 @@
     <inertial>
       <origin xyz="0 0 0" />
-      <mass value="2.8498940e-02" />
-      <inertia ixx="1.1175580e-05" ixy="-4.2369783e-11" ixz="-5.9381719e-09"
-               iyy="1.1192413e-05" iyz="-1.4400107e-11"
-               izz="2.0712558e-05" />
+      <mass value="2.8498940" />
+      <inertia ixx="1.1175580e-03" ixy="-4.2369783e-09" ixz="-5.9381719e-07"
+               iyy="1.1192413e-03" iyz="-1.4400107e-09"
+               izz="2.0712558e-03" />
       </inertial>
   </link>
@@ -139,9 +141,9 @@
     <parent link="base_link"/>
     <child link="base_scan"/>
-    <origin xyz="-0.024 0 0.122" rpy="0 0 0"/>
+    <origin xyz="-0.024 0 0.072" rpy="0 0 0"/>
   </joint>
   <link name="base_scan">
     <visual>
-      <origin xyz="0 0 0.0" rpy="0 0 0"/>
+      <origin xyz="0 0 0.05" rpy="0 0 0"/>
       <geometry>
         <mesh filename="package://turtlebot3_description/meshes/sensors/lds.stl" scale="0.001 0.001 0.001"/>
@@ -150,5 +152,5 @@
     </visual>
     <collision>
-      <origin xyz="0.015 0 -0.0065" rpy="0 0 0"/>
+      <origin xyz="0.015 0 -0.0015" rpy="0 0 0"/>
       <geometry>
         <cylinder length="0.0315" radius="0.045"/>
